File: Node.sch (KiCad schematic (older format))
At the start: 65 parts, among them Q1 NPN

Commit message: fix cpu
Connections:
- wire segments 185 -> 184
Other:
- moved on the sheet: C10, C5, DA2, R2
Changed lines of the file:
@@
 Sheet 1 1
 Title ""
-Date "21 oct 2014"
+Date "29 oct 2014"
 Rev ""
 Comp ""
@@
 Text Notes 13150 2050 0    60   ~ 0
 Matching circuit
-Text Label 5850 1600 0    60   ~ 0
+Text Label 2550 1600 0    60   ~ 0
 CC_GDO2
-Text Label 5850 1700 0    60   ~ 0
+Text Label 2550 1700 0    60   ~ 0
 CC_GDO0
-Text Label 5850 1800 0    60   ~ 0
-CC_CS
 Text Label 5850 1900 0    60   ~ 0
 CC_SCK
@@
 NoConn ~ 5750 3150
 NoConn ~ 5750 3050
-NoConn ~ 5750 2900
 Text Notes 13750 6250 0    60   Italic 12
 Debug port
@@
 Text Label 2950 2200 2    60   ~ 0
 GREEN_LED
-$Comp
-L STM32L151CXTX DD1
-U 1 1 542519DB
-P 4400 2600
-F 0 "DD1" H 3900 3950 60  0000 C CNN
-F 1 "STM32L151CXTX" H 4550 3950 60  0000 C CNN
-F 2 "~" H 4400 2600 60  0000 C CNN
-F 3 "~" H 4400 2600 60  0000 C CNN
-	1    4400 2600
-	1    0    0    -1
-$EndComp
 $Comp
 L LED D2
@@
 L R R2
 U 1 1 542E3AA1
-P 6650 1600
-F 0 "R2" V 6730 1450 50  0000 C CNN
-F 1 "1k" V 6650 1600 50  0000 C CNN
-F 2 "RES_0603" V 6730 1700 28  0000 C CNN
-F 3 "~" H 6650 1600 60  0000 C CNN
-	1    6650 1600
+P 2200 1500
+F 0 "R2" V 2280 1350 50  0000 C CNN
+F 1 "1k" V 2200 1500 50  0000 C CNN
+F 2 "RES_0603" V 2280 1600 28  0000 C CNN
+F 3 "~" H 2200 1500 60  0000 C CNN
+	1    2200 1500
 	0    -1   -1   0
 $EndComp
@@
 L +5V #PWR041
 U 1 1 542E3C99
-P 7000 1600
-F 0 "#PWR041" H 7000 1560 30  0001 C CNN
-F 1 "+5V" H 7080 1630 30  0000 C CNN
-F 2 "~" H 7000 1600 60  0000 C CNN
-F 3 "~" H 7000 1600 60  0000 C CNN
-	1    7000 1600
-	1    0    0    -1
+P 1650 1500
+F 0 "#PWR041" H 1650 1460 30  0001 C CNN
+F 1 "+5V" H 1730 1530 30  0000 C CNN
+F 2 "~" H 1650 1500 60  0000 C CNN
+F 3 "~" H 1650 1500 60  0000 C CNN
+	1    1650 1500
+	-1   0    0    1
 $EndComp
 NoConn ~ 3100 1400
-Text Label 2950 2100 2    60   ~ 0
+Text Label 6250 1700 2    60   ~ 0
 klNFC_Rx
-Text Label 2950 1700 2    60   ~ 0
+Text Label 6600 2900 2    60   ~ 0
 klNFCModulation
 $Comp
@@
 L LD1117 DA2
 U 1 1 543A78F5
-P 4200 6050
-F 0 "DA2" H 4100 6350 60  0000 C CNN
-F 1 "LD1117" H 4200 6250 60  0000 C CNN
-F 2 "~" H 4200 6050 60  0000 C CNN
-F 3 "~" H 4200 6050 60  0000 C CNN
-	1    4200 6050
-	1    0    0    -1
-$EndComp
-Text Label 2950 2000 2    60   ~ 0
+P 5450 6200
+F 0 "DA2" H 5350 6500 60  0000 C CNN
+F 1 "LD1117" H 5450 6400 60  0000 C CNN
+F 2 "~" H 5450 6200 60  0000 C CNN
+F 3 "~" H 5450 6200 60  0000 C CNN
+	1    5450 6200
+	1    0    0    -1
+$EndComp
+Text Label 6250 1500 2    60   ~ 0
 klNFC_Tx
-NoConn ~ 3100 1500
 NoConn ~ 3100 1800
 NoConn ~ 3100 1900
@@
 L +3.3V #PWR060
 U 1 1 543A7B22
-P 5250 6000
-F 0 "#PWR060" H 5250 5960 30  0001 C CNN
-F 1 "+3.3V" H 5330 6030 30  0000 C CNN
-F 2 "~" H 5250 6000 60  0000 C CNN
-F 3 "~" H 5250 6000 60  0000 C CNN
-	1    5250 6000
+P 6500 6150
+F 0 "#PWR060" H 6500 6110 30  0001 C CNN
+F 1 "+3.3V" H 6580 6180 30  0000 C CNN
+F 2 "~" H 6500 6150 60  0000 C CNN
+F 3 "~" H 6500 6150 60  0000 C CNN
+	1    6500 6150
 	1    0    0    -1
 $EndComp
@@
 L GND #PWR061
 U 1 1 543A8018
-P 4200 6800
-F 0 "#PWR061" H 4290 6780 30  0001 C CNN
-F 1 "GND" H 4200 6720 30  0001 C CNN
-F 2 "~" H 4200 6800 60  0000 C CNN
-F 3 "~" H 4200 6800 60  0000 C CNN
-	1    4200 6800
+P 5450 6950
+F 0 "#PWR061" H 5540 6930 30  0001 C CNN
+F 1 "GND" H 5450 6870 30  0001 C CNN
+F 2 "~" H 5450 6950 60  0000 C CNN
+F 3 "~" H 5450 6950 60  0000 C CNN
+	1    5450 6950
 	1    0    0    -1
 $EndComp
@@
 L C C10
 U 1 1 543A8027
-P 5000 6350
-F 0 "C10" H 4900 6250 50  0000 L CNN
-F 1 "u10" H 4900 6450 50  0000 C CNN
-F 2 "CAP_0603" V 5100 6200 28  0000 C BNN
-F 3 "~" H 5000 6350 60  0000 R CNN
-	1    5000 6350
+P 6250 6500
+F 0 "C10" H 6150 6400 50  0000 L CNN
+F 1 "u10" H 6150 6600 50  0000 C CNN
+F 2 "CAP_0603" V 6350 6350 28  0000 C BNN
+F 3 "~" H 6250 6500 60  0000 R CNN
+	1    6250 6500
 	1    0    0    -1
 $EndComp
@@
 	14450 3250 14450 3300
 Wire Wire Line
-	5850 1700 5750 1700
-Wire Wire Line
-	5750 1800 5850 1800
-Wire Wire Line
-	5850 1900 5750 1900
-Wire Wire Line
-	5750 2000 5850 2000
-Wire Wire Line
-	5850 2100 5750 2100
-Wire Wire Line
-	5750 1600 5850 1600
+	5750 1900 6250 1900
+Wire Wire Line
+	5750 2000 6250 2000
+Wire Wire Line
+	5750 2100 6250 2100
+Wire Wire Line
+	5750 1600 6850 1600
 Wire Wire Line
 	12950 2550 11500 2550
@@
 	8250 11200 8350 11200
 Wire Wire Line
-	5750 2300 5850 2300
-Wire Wire Line
-	5750 2400 5850 2400
-Wire Wire Line
-	5750 2500 5850 2500
-Wire Wire Line
-	5750 2600 5850 2600
-Wire Wire Line
-	5750 2700 5850 2700
-Wire Wire Line
-	5750 2800 5850 2800
-Wire Wire Line
-	5750 1500 6400 1500
-Wire Wire Line
-	6400 1500 6400 1600
-Wire Wire Line
-	6900 1600 7000 1600
-Wire Wire Line
-	3100 2100 2950 2100
-Wire Wire Line
-	3100 1700 2050 1700
-Wire Wire Line
-	2050 1700 2050 1600
-Wire Wire Line
-	2050 1600 3100 1600
+	5750 2300 6250 2300
+Wire Wire Line
+	5750 2400 6250 2400
+Wire Wire Line
+	5750 2500 6250 2500
+Wire Wire Line
+	5750 2600 6250 2600
+Wire Wire Line
+	5750 2700 6250 2700
+Wire Wire Line
+	5750 2800 6250 2800
+Wire Wire Line
+	2450 1500 3100 1500
 Wire Wire Line
 	1400 10000 1400 10100
@@
 	1400 9400 1600 9400
 Wire Wire Line
-	3100 2000 2950 2000
-Wire Wire Line
-	4600 6150 4700 6150
-Wire Wire Line
-	4700 6150 4700 6000
-Connection ~ 4700 6000
-Wire Wire Line
-	4200 6800 4200 6400
-Wire Wire Line
-	5000 6800 5000 6550
+	5850 6300 5950 6300
+Wire Wire Line
+	5950 6300 5950 6150
+Connection ~ 5950 6150
+Wire Wire Line
+	5450 6950 5450 6550
+Wire Wire Line
+	6250 6950 6250 6700
 $Comp
 L GND #PWR062
 U 1 1 543A83C7
-P 5000 6800
-F 0 "#PWR062" H 5090 6780 30  0001 C CNN
-F 1 "GND" H 5000 6720 30  0001 C CNN
-F 2 "~" H 5000 6800 60  0000 C CNN
-F 3 "~" H 5000 6800 60  0000 C CNN
-	1    5000 6800
-	1    0    0    -1
-$EndComp
-Wire Wire Line
-	3100 6000 3900 6000
+P 6250 6950
+F 0 "#PWR062" H 6340 6930 30  0001 C CNN
+F 1 "GND" H 6250 6870 30  0001 C CNN
+F 2 "~" H 6250 6950 60  0000 C CNN
+F 3 "~" H 6250 6950 60  0000 C CNN
+	1    6250 6950
+	1    0    0    -1
+$EndComp
+Wire Wire Line
+	4350 6150 5150 6150
 $Comp
 L C C5
 U 1 1 543A85A4
-P 3500 6350
-F 0 "C5" H 3400 6250 50  0000 L CNN
-F 1 "u10" H 3400 6450 50  0000 C CNN
-F 2 "CAP_0603" V 3600 6200 28  0000 C BNN
-F 3 "~" H 3500 6350 60  0000 C CNN
-	1    3500 6350
-	1    0    0    -1
-$EndComp
-Wire Wire Line
-	3500 6550 3500 6800
+P 4750 6500
+F 0 "C5" H 4650 6400 50  0000 L CNN
+F 1 "u10" H 4650 6600 50  0000 C CNN
+F 2 "CAP_0603" V 4850 6350 28  0000 C BNN
+F 3 "~" H 4750 6500 60  0000 C CNN
+	1    4750 6500
+	1    0    0    -1
+$EndComp
+Wire Wire Line
+	4750 6700 4750 6950
 $Comp
 L GND #PWR063
 U 1 1 543A886E
-P 3500 6800
-F 0 "#PWR063" H 3590 6780 30  0001 C CNN
-F 1 "GND" H 3500 6720 30  0001 C CNN
-F 2 "~" H 3500 6800 60  0000 C CNN
-F 3 "~" H 3500 6800 60  0000 C CNN
-	1    3500 6800
-	1    0    0    -1
-$EndComp
-Wire Wire Line
-	4600 6000 5250 6000
-Wire Wire Line
-	5000 6150 5000 6000
-Connection ~ 5000 6000
+P 4750 6950
+F 0 "#PWR063" H 4840 6930 30  0001 C CNN
+F 1 "GND" H 4750 6870 30  0001 C CNN
+F 2 "~" H 4750 6950 60  0000 C CNN
+F 3 "~" H 4750 6950 60  0000 C CNN
+	1    4750 6950
+	1    0    0    -1
+$EndComp
+Wire Wire Line
+	5850 6150 6500 6150
+Wire Wire Line
+	6250 6300 6250 6150
+Connection ~ 6250 6150
 $Comp
 L +5V #PWR064
 U 1 1 543A8A85
-P 3100 6000
-F 0 "#PWR064" H 3100 5960 30  0001 C CNN
-F 1 "+5V" H 3180 6030 30  0000 C CNN
-F 2 "~" H 3100 6000 60  0000 C CNN
-F 3 "~" H 3100 6000 60  0000 C CNN
-	1    3100 6000
+P 4350 6150
+F 0 "#PWR064" H 4350 6110 30  0001 C CNN
+F 1 "+5V" H 4430 6180 30  0000 C CNN
+F 2 "~" H 4350 6150 60  0000 C CNN
+F 3 "~" H 4350 6150 60  0000 C CNN
+	1    4350 6150
 	-1   0    0    1
 $EndComp
@@
 	13400 7950 13500 7950
 Connection ~ 13500 7950
-NoConn ~ 5750 1400
 Connection ~ 3300 9400
 Wire Wire Line
-	3500 6150 3500 6000
-Connection ~ 3500 6000
+	4750 6300 4750 6150
+Connection ~ 4750 6150
 NoConn ~ 3100 2400
 NoConn ~ 3100 2500
+$Comp
+L STM32L151CXTX DD1
+U 1 1 542519DB
+P 4400 2600
+F 0 "DD1" H 3900 3950 60  0000 C CNN
+F 1 "STM32L151CXTX" H 4550 3950 60  0000 C CNN
+F 2 "~" H 4400 2600 60  0000 C CNN
+F 3 "~" H 4400 2600 60  0000 C CNN
+	1    4400 2600
+	1    0    0    -1
+$EndComp
+Wire Wire Line
+	1650 1500 1950 1500
+Wire Wire Line
+	2550 1600 3100 1600
+Wire Wire Line
+	2550 1700 3100 1700
+Wire Wire Line
+	5750 1500 6250 1500
+Wire Wire Line
+	5750 1700 6250 1700
+Wire Wire Line
+	6850 1600 6850 2900
+Wire Wire Line
+	6850 2900 5750 2900
+Text Label 5850 1400 0    60   ~ 0
+CC_CS
+Wire Wire Line
+	5750 1400 6250 1400
+NoConn ~ 3100 2000
+NoConn ~ 3100 2100
+NoConn ~ 5750 1800
 $EndSCHEMATC
